Commit message: 0520

File: model/nezha/urdf/robot_arm.urdf (robot description, URDF)
Before this commit: robot nezha, 24 links, 23 joints
Joints:
- joint left_arm_joint4: limit lower=-2.0 upper=2.0 effort=100 velocity=8 -> lower=-3.14 upper=3.14 effort=100 velocity=8
- joint left_arm_joint6: limit lower=-2.0 upper=2.0 effort=100 velocity=8 -> lower=-3.14 upper=3.14 effort=100 velocity=8
- joint right_arm_joint4: limit lower=-2.0 upper=2.0 effort=0 velocity=0 -> lower=-3.14 upper=3.14 effort=0 velocity=0
- joint right_arm_joint6: limit lower=-2.0 upper=2.0 effort=0 velocity=0 -> lower=-3.14 upper=3.14 effort=0 velocity=0
